Commit message: Finalized URDF of PiDog

File: pidog_description/urdf/pidog.urdf (robot description, URDF)
Before this commit: robot PiDog, 14 links, 13 joints
Links:
- added link back_left_leg_a, mass 0.007296257; collision mesh filename=package://pidog_description/meshes/leg_a.dae; visual mesh filename=package://pidog_description/meshes/leg_a.dae
- added link back_left_leg_b, mass 0.007296257; collision mesh filename=package://pidog_description/meshes/leg_b.dae; visual mesh filename=package://pidog_description/meshes/leg_b.dae
- added link eyes, mass 0.001927895; collision mesh filename=package://pidog_description/meshes/eyes.dae; visual mesh filename=package://pidog_description/meshes/eyes.dae
- added link head, mass 0.001927895; collision mesh filename=package://pidog_description/meshes/head.dae; visual mesh filename=package://pidog_description/meshes/head.dae
- added link motor_10, mass 0.009000000; collision mesh filename=package://pidog_description/meshes/motor.dae; visual mesh filename=package://pidog_description/meshes/motor.dae
- added link motor_11, mass 0.009000000; collision mesh filename=package://pidog_description/meshes/motor.dae; visual mesh filename=package://pidog_description/meshes/motor.dae
- added link motor_6, mass 0.009000000; collision mesh filename=package://pidog_description/meshes/motor.dae; visual mesh filename=package://pidog_description/meshes/motor.dae
- added link motor_7, mass 0.009000000; collision mesh filename=package://pidog_description/meshes/motor.dae; visual mesh filename=package://pidog_description/meshes/motor.dae
- added link motor_8, mass 0.009000000; collision mesh filename=package://pidog_description/meshes/motor.dae; visual mesh filename=package://pidog_description/meshes/motor.dae
- added link motor_9, mass 0.009000000; collision mesh filename=package://pidog_description/meshes/motor.dae; visual mesh filename=package://pidog_description/meshes/motor.dae
- added link neck1, mass 0.001927895; collision mesh filename=package://pidog_description/meshes/neck1.dae; visual mesh filename=package://pidog_description/meshes/neck1.dae
- added link neck2, mass 0.001927895; collision mesh filename=package://pidog_description/meshes/neck2.dae; visual mesh filename=package://pidog_description/meshes/neck2.dae
- added link neck3, mass 0.001927895; collision mesh filename=package://pidog_description/meshes/neck3.dae; visual mesh filename=package://pidog_description/meshes/neck3.dae
Joints:
- removed joint body_to_from_left_leg_b
- removed joint body_to_tail
- removed joint front_left_leg_a_to_motor_5
- removed joint front_left_leg_b_to_motor_4
- added joint back_left_leg_a_to_motor_5: type fixed, parent back_left_leg_a, child motor_5, origin xyz=0 0 0 rpy=0 0 0
- added joint back_left_leg_b_to_a: type revolute, parent back_left_leg_b, child back_left_leg_a, origin xyz=0.047 0 0.0095 rpy=0 0 1.57, axis 0 0 1, limit lower=-1.57 upper=1.57 effort=0.3 velocity=1.0
- added joint back_left_leg_b_to_motor_4: type fixed, parent back_left_leg_b, child motor_4, origin xyz=0 0 0 rpy=0 0 0
- added joint body_to_back_left_leg_b: type revolute, parent body, child back_left_leg_b, origin xyz=-0.0405 -0.06685 -0.009 rpy=0 1.57 3.1415, axis 0 0 1, limit lower=-1.57 upper=1.57 effort=0.3 velocity=1.0
- added joint body_to_front_left_leg_b: type revolute, parent body, child front_left_leg_b, origin xyz=-0.0405 0.05315 -0.009 rpy=0 1.57 3.1415, axis 0 0 1, limit lower=-1.57 upper=1.57 effort=0.3 velocity=1.0
- added joint body_to_motor_8: type fixed, parent body, child motor_8, origin xyz=0 -0.07375 0.01 rpy=0.785375 0 0
- added joint body_to_neck1: type fixed, parent body, child neck1, origin xyz=0 0.07 0.013 rpy=0 0.785375 1.57075
- added joint front_left_leg_a_to_motor_7: type fixed, parent front_left_leg_a, child motor_7, origin xyz=0 0 0 rpy=0 0 0
- added joint front_left_leg_b_to_motor_6: type fixed, parent front_left_leg_b, child motor_6, origin xyz=0 0 0 rpy=0 0 0
- added joint head_to_eyes: type fixed, parent head, child eyes, origin xyz=0.0 0.0 0.036 rpy=0 0.0 0
- added joint motor_10_to_neck3: type fixed, parent motor_10, child neck3, origin xyz=0.011 0.0 -0.0 rpy=0.0 0.0 0.0
- added joint motor_11_to_head: type fixed, parent motor_11, child head, origin xyz=0.025 0.0 0.015 rpy=0 0.0 0
- added joint motor_8_to_tail: type revolute, parent motor_8, child tail, origin xyz=0 0 0.008 rpy=0 0 0, axis 0 0 1, limit lower=-1.57 upper=1.57 effort=0.3 velocity=1.0
- added joint motor_9_to_neck2: type fixed, parent motor_9, child neck2, origin xyz=0.006 -0.001 0.0125 rpy=0.0 0.0 0.0
- added joint neck1_to_motor_9: type revolute, parent neck1, child motor_9, origin xyz=0 0.01 0.015 rpy=1.57075 0.785375 0, axis 0 0 1, limit lower=-1.57 upper=1.57 effort=0.3 velocity=1.0
- added joint neck2_to_motor_10: type revolute, parent neck2, child motor_10, origin xyz=0 -0.021 -0.003 rpy=-1.57075 0 3.1415, axis 0 0 1, limit lower=-1.57 upper=1.57 effort=0.3 velocity=1.0
- added joint neck3_to_motor_11: type revolute, parent neck3, child motor_11, origin xyz=0.0265 0.0 -0.0125 rpy=0 1.57075 0, axis 0 0 1, limit lower=-1.57 upper=1.57 effort=0.3 velocity=1.0
- joint body_to_back_right_leg_b: origin xyz=0.04075 -0.07575 -0.009 rpy=0 1.57 0 -> xyz=0.0405 -0.06685 -0.009 rpy=0 1.57 0
- joint body_to_from_right_leg_b: origin xyz=0.04075 0.04425 -0.009 rpy=0 1.57 0 -> xyz=0.0405 0.05315 -0.009 rpy=0 1.57 0

Commit message: Finalized URDF

File: pidog_description/urdf/pidog.urdf (robot description, URDF)
Before this commit: robot PiDog, 27 links, 26 joints
Links:
- added link back_left_acrylic, mass 0.00316; collision mesh filename=package://pidog_description/meshes/acrylic.dae; visual mesh filename=package://pidog_description/meshes/acrylic.dae
- added link back_right_acrylic, mass 0.00316; collision mesh filename=package://pidog_description/meshes/acrylic.dae; visual mesh filename=package://pidog_description/meshes/acrylic.dae
- added link front_left_acrylic, mass 0.00316; collision mesh filename=package://pidog_description/meshes/acrylic.dae; visual mesh filename=package://pidog_description/meshes/acrylic.dae
- added link front_right_acrylic, mass 0.00316; collision mesh filename=package://pidog_description/meshes/acrylic.dae; visual mesh filename=package://pidog_description/meshes/acrylic.dae
Joints:
- added joint back_left_leg_a_to_acrylic: type fixed, parent back_left_leg_a, child back_left_acrylic, origin xyz=-0.0635 -0.00225 -0.001 rpy=0 0 0
- added joint back_right_leg_a_to_acrylic: type fixed, parent back_right_leg_a, child back_right_acrylic, origin xyz=0.0635 -0.00225 0.001 rpy=0 3.1415 0
- added joint front_left_leg_a_to_acrylic: type fixed, parent front_left_leg_a, child front_left_acrylic, origin xyz=-0.0635 -0.00225 -0.001 rpy=0 0 0
- added joint front_right_leg_a_to_acrylic: type fixed, parent front_right_leg_a, child front_right_acrylic, origin xyz=0.0635 -0.00225 0.001 rpy=0 3.1415 0

Commit message: Started woking on the webots simulator

File: pidog_description/urdf/pidog.urdf (robot description, URDF)
Before this commit: robot PiDog, 31 links, 30 joints
Links:
- link eyes: mass 0.001927895 -> 0.036527618
- link head: mass 0.001927895 -> 0.045943792
- link neck2: mass 0.001927895 -> 0.008369068
- link neck3: mass 0.001927895 -> 0.008817173
Joints:
- joint back_left_leg_b_to_a: limit lower=-1.57 upper=1.57 effort=0.3 velocity=1.0 -> lower=-1.57 upper=1.57 effort=0.3
- joint back_right_leg_b_to_a: limit lower=-1.57 upper=1.57 effort=0.3 velocity=1.0 -> lower=-1.57 upper=1.57 effort=0.3
- joint body_to_back_left_leg_b: limit lower=-1.57 upper=1.57 effort=0.3 velocity=1.0 -> lower=-1.57 upper=1.57 effort=0.3
- joint body_to_back_right_leg_b: limit lower=-1.57 upper=1.57 effort=0.3 velocity=1.0 -> lower=-1.57 upper=1.57 effort=0.3
- joint body_to_from_right_leg_b: limit lower=-1.57 upper=1.57 effort=0.3 velocity=1.0 -> lower=-1.57 upper=1.57 effort=0.3
- joint body_to_front_left_leg_b: limit lower=-1.57 upper=1.57 effort=0.3 velocity=1.0 -> lower=-1.57 upper=1.57 effort=0.3
- joint front_left_leg_b_to_a: limit lower=-1.57 upper=1.57 effort=0.3 velocity=1.0 -> lower=-1.57 upper=1.57 effort=0.3
- joint front_right_leg_b_to_a: limit lower=-1.57 upper=1.57 effort=0.3 velocity=1.0 -> lower=-1.57 upper=1.57 effort=0.3
- joint motor_8_to_tail: limit lower=-1.57 upper=1.57 effort=0.3 velocity=1.0 -> lower=-1.57 upper=1.57 effort=0.3
- joint neck1_to_motor_9: limit lower=-1.57 upper=1.57 effort=0.3 velocity=1.0 -> lower=-1.57 upper=1.57 effort=0.3
- joint neck2_to_motor_10: limit lower=-1.57 upper=1.57 effort=0.3 velocity=1.0 -> lower=-1.57 upper=1.57 effort=0.3
- joint neck3_to_motor_11: limit lower=-1.57 upper=1.57 effort=0.3 velocity=1.0 -> lower=-1.57 upper=1.57 effort=0.3

Commit message: Created a script to test cross machine communication

File: pidog_description/urdf/pidog.urdf (robot description, URDF)
Before this commit: robot PiDog, 31 links, 30 joints
Joints:
- removed joint body_to_from_right_leg_b
- added joint body_to_front_right_leg_b: type revolute, parent body, child front_right_leg_b, origin xyz=0.0405 0.05315 -0.009 rpy=1.57 0 1.57, axis 0 0 1, limit lower=-1.57 upper=1.57 effort=0.3 velocity=10.0
- joint back_left_leg_a_to_acrylic: origin xyz=-0.0635 -0.00225 -0.001 rpy=0 0 0 -> xyz=0.00225 -0.0635 -0.001 rpy=0 0 1.57
- joint back_left_leg_b_to_a: limit lower=-1.57 upper=1.57 effort=0.3 -> lower=-1.57 upper=1.57 effort=0.3 velocity=10.0; origin xyz=0.047 0 0.0095 rpy=0 0 1.57 -> xyz=0.0 0.047 0.0095 rpy=0 0 1.57
- joint back_right_leg_a_to_acrylic: origin xyz=0.0635 -0.00225 0.001 rpy=0 3.1415 0 -> xyz=0.00225 0.0635 0.001 rpy=0 3.1415 1.57
- joint back_right_leg_b_to_a: limit lower=-1.57 upper=1.57 effort=0.3 -> lower=-1.57 upper=1.57 effort=0.3 velocity=10.0; origin xyz=0.047 0 0.0095 rpy=0 0 1.57 -> xyz=0 -0.047 0.0095 rpy=0 0 -1.57
- joint body_to_back_left_leg_b: limit lower=-1.57 upper=1.57 effort=0.3 -> lower=-1.57 upper=1.57 effort=0.3 velocity=10.0; origin xyz=-0.0405 -0.06685 -0.009 rpy=0 1.57 3.1415 -> xyz=-0.0405 -0.06685 -0.009 rpy=-1.57 0 1.57
- joint body_to_back_right_leg_b: limit lower=-1.57 upper=1.57 effort=0.3 -> lower=-1.57 upper=1.57 effort=0.3 velocity=10.0; origin xyz=0.0405 -0.06685 -0.009 rpy=0 1.57 0 -> xyz=0.0405 -0.06685 -0.009 rpy=1.57 0 1.57
- joint body_to_front_left_leg_b: limit lower=-1.57 upper=1.57 effort=0.3 -> lower=-1.57 upper=1.57 effort=0.3 velocity=10.0; origin xyz=-0.0405 0.05315 -0.009 rpy=0 1.57 3.1415 -> xyz=-0.0405 0.05315 -0.009 rpy=-1.57 0 1.57
- joint front_left_leg_a_to_acrylic: origin xyz=-0.0635 -0.00225 -0.001 rpy=0 0 0 -> xyz=0.00225 -0.0635 -0.001 rpy=0 0 1.57
- joint front_left_leg_b_to_a: limit lower=-1.57 upper=1.57 effort=0.3 -> lower=-1.57 upper=1.57 effort=0.3 velocity=10.0; origin xyz=0.047 0 0.0095 rpy=0 0 1.57 -> xyz=0.0 0.047 0.0095 rpy=0 0 1.57
- joint front_right_leg_a_to_acrylic: origin xyz=0.0635 -0.00225 0.001 rpy=0 3.1415 0 -> xyz=0.00225 0.0635 0.001 rpy=0 3.1415 1.57
- joint front_right_leg_b_to_a: limit lower=-1.57 upper=1.57 effort=0.3 -> lower=-1.57 upper=1.57 effort=0.3 velocity=10.0; origin xyz=0.047 0 0.0095 rpy=0 0 1.57 -> xyz=0 -0.047 0.0095 rpy=0 0 -1.57
- joint motor_8_to_tail: limit lower=-1.57 upper=1.57 effort=0.3 -> lower=-1.57 upper=1.57 effort=0.3 velocity=10.0
- joint neck1_to_motor_9: limit lower=-1.57 upper=1.57 effort=0.3 -> lower=-1.57 upper=1.57 effort=0.3 velocity=10.0
- joint neck2_to_motor_10: limit lower=-1.57 upper=1.57 effort=0.3 -> lower=-1.57 upper=1.57 effort=0.3 velocity=10.0
- joint neck3_to_motor_11: limit lower=-1.57 upper=1.57 effort=0.3 -> lower=-1.57 upper=1.57 effort=0.3 velocity=10.0
